Commit message: updated URDF

File: bevy_sim_urdf/assets/urdf/urdf_assembly.urdf (robot description, URDF)
Before this commit: robot urdf_assembly, 125 links, 124 joints
Links:
- removed link camera_dsj_3808_308
- removed link cup_point_hex_socket_set_screw_m3x0_5_x_3
- removed link cup_point_hex_socket_set_screw_m3x0_5_x_3_1
- removed link cup_point_hex_socket_set_screw_m3x0_5_x_5
- removed link ethercat_subdevice_pcb_3d_1__1_
- removed link flangedbearing5mm
- removed link flangedbearing5mm_1
- removed link flangedbearing5mm_10
- removed link flangedbearing5mm_11
- removed link flangedbearing5mm_2
- removed link flangedbearing5mm_3
- removed link flangedbearing5mm_4
- removed link flangedbearing5mm_5
- removed link flangedbearing5mm_6
- removed link flangedbearing5mm_7
- removed link flangedbearing5mm_8
- removed link flangedbearing5mm_9
- removed link flat_point_hex_socket_set_screw_m3x0_5_x_4
- removed link hex_nut_grade_a___b_m3x0_5
- removed link hex_nut_grade_a___b_m3x0_5_1
- removed link hex_nut_grade_a___b_m3x0_5_10
- removed link hex_nut_grade_a___b_m3x0_5_11
- removed link hex_nut_grade_a___b_m3x0_5_12
- removed link hex_nut_grade_a___b_m3x0_5_13
- removed link hex_nut_grade_a___b_m3x0_5_2
- removed link hex_nut_grade_a___b_m3x0_5_3
- removed link hex_nut_grade_a___b_m3x0_5_4
- removed link hex_nut_grade_a___b_m3x0_5_5
- removed link hex_nut_grade_a___b_m3x0_5_6
- removed link hex_nut_grade_a___b_m3x0_5_7
- removed link hex_nut_grade_a___b_m3x0_5_8
- removed link hex_nut_grade_a___b_m3x0_5_9
- removed link hex_nut_grade_a___b_m4x0_7
- removed link hex_nut_grade_a___b_m4x0_7_1
- removed link hex_nut_grade_a___b_m4x0_7_2
- removed link hex_nut_grade_a___b_m4x0_7_3
- removed link hex_socket_head_cap_screw_m3x0_50_x_12
- removed link hex_socket_head_cap_screw_m3x0_50_x_12_1
- removed link hex_socket_head_cap_screw_m3x0_50_x_12_2
- removed link hex_socket_head_cap_screw_m3x0_50_x_12_3
- removed link hex_socket_head_cap_screw_m3x0_50_x_16
- removed link hex_socket_head_cap_screw_m3x0_50_x_16_1
- removed link hex_socket_head_cap_screw_m3x0_50_x_16_2
- removed link hex_socket_head_cap_screw_m3x0_50_x_16_3
- removed link hex_socket_head_cap_screw_m3x0_50_x_20
- removed link hex_socket_head_cap_screw_m3x0_50_x_20_1
- removed link hex_socket_head_cap_screw_m3x0_50_x_20_2
- removed link hex_socket_head_cap_screw_m3x0_50_x_20_3
- removed link hex_socket_head_cap_screw_m3x0_50_x_20_4
- removed link hex_socket_head_cap_screw_m3x0_50_x_20_5
- removed link jawlinkage
- removed link jawlinkage_1
- removed link motor
- removed link motor_l_bracket
- removed link motorcap
- removed link mountinghub5mmshaft
- removed link mountinghub5mmshaft_1
- removed link shaft5mm
- removed link shaft5mm_1
- removed link shaft5mm_2
- removed link shaft5mm_3
- removed link shoulderscrew
- removed link shoulderscrew_1
- removed link shoulderscrew_2
- removed link shoulderscrew_3
- removed link spacer5x8x17
- removed link spacer5x8x2_5
- removed link spacer5x8x2_5_1
- removed link spacer5x8x2_5_2
- removed link spacer5x8x2_5_3
- removed link spacer5x8x32_5
- removed link spacer5x8x32_5_1
- removed link spacer5x8x5
- removed link spur_gear_l__33_teeth_
- removed link spur_gear_r__33_teeth_
- removed link wormgear
- removed link wormgearspacer
- removed link wormwheel
- added link end_effector_mini_verson__1_
- link erob70f__i_f_xx_18cx_v3_mc2a_9x_xx: mass 2.9591e-05 -> 1.46394e-07
- link erob70f__i_f_xx_18cx_v3_mc2a_9x_xx_2: mass 1.46394e-07 -> 2.9591e-05
- link erob70f__i_f_xx_18cx_v3_mc2a_9x_xx_3: mass 1.46394e-07 -> 0.000156301
- link erob70f__i_f_xx_18cx_v3_mc2a_9x_xx_5: mass 0.000156301 -> 1.46394e-07
- link erob70f__i_f_xx_18cx_v3_mc2a_9x_xx_7: mass 2.9591e-05 -> 0.000156301
- link erob70f__i_f_xx_18cx_v3_mc2a_9x_xx_8: mass 0.000156301 -> 2.9591e-05
- link part_1: mass 3.48219e-05 -> 5.29798e-05
- link part_1_1: mass 2.08777e-05 -> 3.48219e-05
- link part_1_2: mass 2.59613e-05 -> 2.08777e-05
- link part_1_4: mass 5.29798e-05 -> 2.59613e-05
Joints:
- removed joint group_1_fastened_joint
- removed joint group_1_fastened_joint_1
- removed joint group_1_fastened_joint_10
- removed joint group_1_fastened_joint_11
- removed joint group_1_fastened_joint_12
- removed joint group_1_fastened_joint_13
- removed joint group_1_fastened_joint_14
- removed joint group_1_fastened_joint_15
- removed joint group_1_fastened_joint_16
- removed joint group_1_fastened_joint_17
- removed joint group_1_fastened_joint_18
- removed joint group_1_fastened_joint_19
- removed joint group_1_fastened_joint_2
- removed joint group_1_fastened_joint_20
- removed joint group_1_fastened_joint_21
- removed joint group_1_fastened_joint_22
- removed joint group_1_fastened_joint_23
- removed joint group_1_fastened_joint_24
- removed joint group_1_fastened_joint_25
- removed joint group_1_fastened_joint_26
- removed joint group_1_fastened_joint_27
- removed joint group_1_fastened_joint_28
- removed joint group_1_fastened_joint_29
- removed joint group_1_fastened_joint_3
- removed joint group_1_fastened_joint_30
- removed joint group_1_fastened_joint_31
- removed joint group_1_fastened_joint_32
- removed joint group_1_fastened_joint_33
- removed joint group_1_fastened_joint_34
- removed joint group_1_fastened_joint_35
- removed joint group_1_fastened_joint_36
- removed joint group_1_fastened_joint_37
- removed joint group_1_fastened_joint_38
- removed joint group_1_fastened_joint_39
- removed joint group_1_fastened_joint_4
- removed joint group_1_fastened_joint_40
- removed joint group_1_fastened_joint_41
- removed joint group_1_fastened_joint_42
- removed joint group_1_fastened_joint_43
- removed joint group_1_fastened_joint_44
- removed joint group_1_fastened_joint_45
- removed joint group_1_fastened_joint_46
- removed joint group_1_fastened_joint_47
- removed joint group_1_fastened_joint_48
- removed joint group_1_fastened_joint_49
- removed joint group_1_fastened_joint_5
- removed joint group_1_fastened_joint_50
- removed joint group_1_fastened_joint_51
- removed joint group_1_fastened_joint_52
- removed joint group_1_fastened_joint_53
- removed joint group_1_fastened_joint_54
- removed joint group_1_fastened_joint_55
- removed joint group_1_fastened_joint_56
- removed joint group_1_fastened_joint_57
- removed joint group_1_fastened_joint_58
- removed joint group_1_fastened_joint_59
- removed joint group_1_fastened_joint_6
- removed joint group_1_fastened_joint_60
- removed joint group_1_fastened_joint_61
- removed joint group_1_fastened_joint_62
- removed joint group_1_fastened_joint_63
- removed joint group_1_fastened_joint_64
- removed joint group_1_fastened_joint_65
- removed joint group_1_fastened_joint_66
- removed joint group_1_fastened_joint_67
- removed joint group_1_fastened_joint_68
- removed joint group_1_fastened_joint_69
- removed joint group_1_fastened_joint_7
- removed joint group_1_fastened_joint_70
- removed joint group_1_fastened_joint_71
- removed joint group_1_fastened_joint_72
- removed joint group_1_fastened_joint_73
- removed joint group_1_fastened_joint_74
- removed joint group_1_fastened_joint_75
- removed joint group_1_fastened_joint_76
- removed joint group_1_fastened_joint_77
- removed joint group_1_fastened_joint_78
- removed joint group_1_fastened_joint_79
- removed joint group_1_fastened_joint_8
- removed joint group_1_fastened_joint_80
- removed joint group_1_fastened_joint_81
- removed joint group_1_fastened_joint_82
- removed joint group_1_fastened_joint_83
- removed joint group_1_fastened_joint_84
- removed joint group_1_fastened_joint_85
- removed joint group_1_fastened_joint_86
- removed joint group_1_fastened_joint_9
- added joint fastened_10: type fixed, parent fixingwall, child end_effector_mini_verson__1_, origin xyz=-6.93889e-17 -1.11022e-16 -1.56125e-17 rpy=1.5708 -3.22447e-29 -3.14159, axis 0 0 1
- added joint fastened_1_8: type fixed, parent link5base, child link5attachments, origin xyz=-0.0457966 -0.009 -0.01 rpy=-1.5708 -9.73666e-14 1.5708, axis 0 -1 0
- added joint fastened_2_7: type fixed, parent link5base, child link5attachments_1, origin xyz=0.0457966 -0.009 -0.01 rpy=-1.5708 -9.73666e-14 1.5708, axis 0 -1 0
- added joint fastened_3_4: type fixed, parent link5attachments_1, child link5, origin xyz=-0.00330299 0.018 7.99361e-15 rpy=8.63884e-14 1.5584e-14 1.5708, axis 0 -1 0
- added joint fastened_4_3: type fixed, parent part_1_4, child part_1_3, origin xyz=-0.025 -0.0044 0.021 rpy=-1.5708 -7.64881e-14 -4.901e-14, axis -0 -0 1
- added joint fastened_5_5: type fixed, parent link5, child v5, origin xyz=-9.97813e-15 1.70048e-06 0.181211 rpy=0 1.5708 3.14159, axis 0 -1 -6.93889e-16
- added joint fastened_6_2: type fixed, parent v5, child erob70f__i_f_xx_18cx_v3_mc2a_9x_xx_7, origin xyz=-0.0015 0.0349045 0.0313726 rpy=-4.30211e-16 3.27149e-17 -3.33067e-16, axis -1 -4.10789e-17 4.10789e-17
- added joint fastened_7_1: type fixed, parent link5base, child j6_clean_assembly__1_, origin xyz=1.11022e-15 -1.94289e-16 -0.005 rpy=4.33681e-19 -0 0, axis -0 -0 -1
- added joint fastened_8: type fixed, parent cranklinkage, child rockerlinkage_1, origin xyz=0 -0.06 2.1684e-17 rpy=1.65666e-19 -6.26108e-21 1.5708, axis -0 -0 -1
- added joint fastened_9: type fixed, parent lidplate, child cranklinkage, origin xyz=0.01551 -0.092697 -0.045 rpy=-3.14159 3.92174e-19 -1.22173, axis 0 0 1
- joint fastened_1: child erob80h__i_xx_18ex_v6_mc2e_dx_xx_1 -> erob80h__i_xx_18ex_v6_mc2e_dx_xx_2
- joint fastened_1_2: child erob70f__i_f_xx_18cx_v3_mc2a_9x_xx_3 -> erob70f__i_f_xx_18cx_v3_mc2a_9x_xx; parent erob70f__i_f_xx_18cx_v3_mc2a_9x_xx_4 -> erob70f__i_f_xx_18cx_v3_mc2a_9x_xx_2
- joint fastened_1_3: axis -1 1.96285e-16 2.78443e-16 -> -0 -1 -0; child erob70f__i_f_xx_18cx_v3_mc2a_9x_xx_1 -> baseplate; origin xyz=-0.0166838 -0.0110658 -0.0183117 rpy=0 -1.5708 -4.71239 -> xyz=5.55112e-17 -0.0194 -0.0223622 rpy=1.26218e-29 -3.06516e-29 -3.14159; parent motor5housing_1 -> fixingwall
- joint fastened_1_4: axis 1 -1.56367e-16 -2.38525e-16 -> -1 1.96285e-16 2.78443e-16; child erob70f__i_f_xx_18cx_v3_mc2a_9x_xx_2 -> erob70f__i_f_xx_18cx_v3_mc2a_9x_xx_3; origin xyz=-0.00767132 6.93889e-17 7.43849e-15 rpy=-7.88861e-30 -2.52435e-29 5.46438e-17 -> xyz=-0.0166838 -0.0110658 -0.0183117 rpy=0 -1.5708 -4.71239; parent erob70f__i_f_xx_18cx_v3_mc2a_9x_xx -> motor5housing_1
- joint fastened_1_5: axis 1 -0 -0 -> 1 -1.56367e-16 -2.38525e-16; child erob80h__i_xx_18ex_v6_mc2e_dx_xx_2 -> erob70f__i_f_xx_18cx_v3_mc2a_9x_xx_5; origin xyz=0.0095763 0.015 0.0866199 rpy=-3.14159 9.91702e-15 1.5708 -> xyz=-0.00767132 6.93889e-17 7.43849e-15 rpy=-7.88861e-30 -2.52435e-29 5.46438e-17; parent armjoint3mount_final_v4 -> erob70f__i_f_xx_18cx_v3_mc2a_9x_xx_4
- joint fastened_1_6: axis 1 -1.56367e-16 -2.38525e-16 -> 1 -0 -0; child erob70f__i_f_xx_18cx_v3_mc2a_9x_xx_6 -> erob80h__i_xx_18ex_v6_mc2e_dx_xx_1; origin xyz=-0.00767132 1.13798e-15 7.24421e-15 rpy=4.33681e-19 -0 0 -> xyz=0.0095763 0.015 0.0866199 rpy=-3.14159 9.91702e-15 1.5708; parent erob70f__i_f_xx_18cx_v3_mc2a_9x_xx_7 -> armjoint3mount_final_v4
- joint fastened_1_7: axis 0 -1 0 -> 1 -1.56367e-16 -2.38525e-16; child link5attachments -> erob70f__i_f_xx_18cx_v3_mc2a_9x_xx_6; origin xyz=-0.0457966 -0.009 -0.01 rpy=-1.5708 -9.73666e-14 1.5708 -> xyz=-0.00767132 1.13798e-15 7.24421e-15 rpy=4.33681e-19 -0 0; parent link5base -> erob70f__i_f_xx_18cx_v3_mc2a_9x_xx_8
- joint fastened_2_1: child erob70f__i_f_xx_18cx_v3_mc2a_9x_xx_4 -> erob70f__i_f_xx_18cx_v3_mc2a_9x_xx_2; parent erob70f__i_f_xx_18cx_v3_mc2a_9x_xx_5 -> erob70f__i_f_xx_18cx_v3_mc2a_9x_xx_1
- joint fastened_2_2: axis 1 4.66648e-16 -5.37364e-16 -> -0 -0 -1; child erob70f__i_f_xx_18cx_v3_mc2a_9x_xx -> gripperl; origin xyz=0.0155004 3.46551e-08 0.031999 rpy=5.20648e-29 1.00974e-28 -9.36751e-17 -> xyz=-0.005 0.113 0.0024 rpy=-2.28243e-17 -4.61254e-17 1.11022e-16; parent erob70f__i_f_xx_18cx_v3_mc2a_9x_xx_1 -> rockerlinkage_1
- joint fastened_2_3: axis 0 1 0 -> 1 4.66648e-16 -5.37364e-16; child motor5housing_1 -> erob70f__i_f_xx_18cx_v3_mc2a_9x_xx_4; origin xyz=-0.0127279 0.0127279 -0.015 rpy=1.5708 5.55112e-16 1.9635 -> xyz=0.0155004 3.46551e-08 0.031999 rpy=5.20648e-29 1.00974e-28 -9.36751e-17; parent part_1_1 -> erob70f__i_f_xx_18cx_v3_mc2a_9x_xx_3
- joint fastened_2_4: axis -0 -0 -1 -> 0 1 0; child armjoint3mount_final_v4 -> motor5housing_1; origin xyz=-2.88658e-15 3.84415e-15 0.22 rpy=-1.30398e-15 -8.9026e-15 -8.74349e-15 -> xyz=-0.0127279 0.0127279 -0.015 rpy=1.5708 5.55112e-16 1.9635; parent part_1_3 -> part_1_2
- joint fastened_2_5: axis 1 4.66648e-16 -5.37364e-16 -> -0 -0 -1; child erob70f__i_f_xx_18cx_v3_mc2a_9x_xx_7 -> armjoint3mount_final_v4; origin xyz=0.0155 -0.0226274 0.0226274 rpy=-1.60462e-17 3.92231e-16 7.21645e-16 -> xyz=-2.88658e-15 3.84415e-15 0.22 rpy=-1.30398e-15 -8.9026e-15 -8.74349e-15; parent erob70f__i_f_xx_18cx_v3_mc2a_9x_xx_8 -> part_1_3
- joint fastened_2_6: axis 0 -1 0 -> 1 4.66648e-16 -5.37364e-16; child link5attachments_1 -> erob70f__i_f_xx_18cx_v3_mc2a_9x_xx_8; origin xyz=0.0457966 -0.009 -0.01 rpy=-1.5708 -9.73666e-14 1.5708 -> xyz=0.0155 -0.0226274 0.0226274 rpy=-1.60462e-17 3.92231e-16 7.21645e-16; parent link5base -> erob70f__i_f_xx_18cx_v3_mc2a_9x_xx_7
- joint fastened_3: axis 0 0 1 -> -0 -0 1; child part_1_1 -> gripperr; origin xyz=-2.42861e-17 -5.55112e-17 0.225 rpy=3.14159 6.31089e-30 -3.14159 -> xyz=-0.005 0.113 -0.0076 rpy=-6.34311e-19 8.313e-17 5.55112e-17; parent link4 -> rockerlinkage
- joint fastened_3_1: axis -0 -0 -1 -> 0 0 1; origin xyz=0.024979 -0.01568 0.01 rpy=-2.26019e-14 -2.85422e-14 1.60635e-14 -> xyz=-2.42861e-17 -5.55112e-17 0.225 rpy=3.14159 6.31089e-30 -3.14159; parent armjoint2rotor_final_v2 -> link4
- joint fastened_3_2: axis 1 0 0 -> -0 -0 -1; child erob80h__i_xx_18ex_v6_mc2e_dx_xx -> part_1_4; origin xyz=0.00575166 -0.0882991 0.00863101 rpy=0 -1.5708 -1.5708 -> xyz=0.024979 -0.01568 0.01 rpy=-2.26019e-14 -2.85422e-14 1.60635e-14; parent motor5housing -> armjoint2rotor_final_v2
- joint fastened_3_3: axis 0 -1 0 -> 1 0 0; child link5 -> erob80h__i_xx_18ex_v6_mc2e_dx_xx; origin xyz=-0.00330299 0.018 7.99361e-15 rpy=8.63884e-14 1.5584e-14 1.5708 -> xyz=0.00575166 -0.0882991 0.00863101 rpy=0 -1.5708 -1.5708; parent link5attachments_1 -> motor5housing
- joint fastened_4: child part_1_4 -> part_1
- joint fastened_4_1: axis 0 0 -1 -> -1 0 -2.77556e-16; child link4 -> lidplate; origin xyz=-1.9082e-17 3.46945e-17 0.013 rpy=-1.38778e-16 -1.85961e-16 2.22045e-16 -> xyz=-3.46945e-17 0.129697 -0.00625547 rpy=3.14159 -4.17201e-16 -3.14159; parent link4bottomattachment -> baseplate
- joint fastened_4_2: axis -0 -0 1 -> 0 0 -1; child part_1_3 -> link4; origin xyz=-0.025 -0.0044 0.021 rpy=-1.5708 -7.64881e-14 -4.901e-14 -> xyz=-1.9082e-17 3.46945e-17 0.013 rpy=-1.38778e-16 -1.85961e-16 2.22045e-16; parent part_1_2 -> link4bottomattachment
- joint fastened_5: parent part_1_4 -> part_1
- joint fastened_5_1: axis -0 -0 1 -> -0 -0 -1; child j5_wrist_pitch_copy_1__1_ -> rockerlinkage; origin xyz=-2.08167e-17 6.93889e-18 -2.22045e-16 rpy=6.31089e-30 6.31089e-30 3.14159 -> xyz=0 -0.06 0.005 rpy=-9.4475e-17 1.0642e-16 1.5708; parent link4bottomattachment -> cranklinkage_1
- joint fastened_5_2: axis 0 0 1 -> -0 -0 1; child j3_new_assembly__1_ -> j5_wrist_pitch_copy_1__1_; origin xyz=-8.11851e-16 -0.04 1.10328e-15 rpy=-1.5708 -1.91513e-14 1.5708 -> xyz=-2.08167e-17 6.93889e-18 -2.22045e-16 rpy=6.31089e-30 6.31089e-30 3.14159; parent armjoint2rotor_final_v2 -> link4bottomattachment
- joint fastened_5_3: axis -1.25497e-16 1 0 -> 0 0 1; child motor5housing -> j3_new_assembly__1_; origin xyz=0.0153343 -0.00646891 0.041 rpy=-1.5708 1.15024e-15 -3.14159 -> xyz=-8.11851e-16 -0.04 1.10328e-15 rpy=-1.5708 -1.91513e-14 1.5708; parent part_1 -> armjoint2rotor_final_v2
- joint fastened_5_4: axis 0 -1 -6.93889e-16 -> -1.25497e-16 1 0; child v5 -> motor5housing; origin xyz=-9.97813e-15 1.70048e-06 0.181211 rpy=0 1.5708 3.14159 -> xyz=0.0153343 -0.00646891 0.041 rpy=-1.5708 1.15024e-15 -3.14159; parent link5 -> part_1_1
- joint fastened_6: child erob70f__i_f_xx_18cx_v3_mc2a_9x_xx_5 -> erob70f__i_f_xx_18cx_v3_mc2a_9x_xx_1; parent part_1_4 -> part_1
- joint fastened_6_1: axis -1 -4.10789e-17 4.10789e-17 -> 0 0 -1; child erob70f__i_f_xx_18cx_v3_mc2a_9x_xx_8 -> cranklinkage_1; origin xyz=-0.0015 0.0349045 0.0313726 rpy=-4.30211e-16 3.27149e-17 -3.33067e-16 -> xyz=-0.01551 -0.092697 -0.045 rpy=-1.44514e-16 -3.5339e-18 -1.91986; parent v5 -> lidplate
- joint fastened_7: axis -0 -0 -1 -> 1 -5.63222e-17 0; child j6_clean_assembly__1_ -> motorhousing; origin xyz=1.11022e-15 -1.94289e-16 -0.005 rpy=4.33681e-19 -0 0 -> xyz=-0.01645 0.0555 0.00604453 rpy=1.26598e-29 -4.50161e-16 -1.68967e-16; parent link5base -> baseplate
- joint revolute_1: child part_1 -> part_1_1; parent erob80h__i_xx_18ex_v6_mc2e_dx_xx_1 -> erob80h__i_xx_18ex_v6_mc2e_dx_xx_2
- joint revolute_3: parent erob80h__i_xx_18ex_v6_mc2e_dx_xx_2 -> erob80h__i_xx_18ex_v6_mc2e_dx_xx_1
- joint revolute_4: parent erob70f__i_f_xx_18cx_v3_mc2a_9x_xx_4 -> erob70f__i_f_xx_18cx_v3_mc2a_9x_xx_2
- joint revolute_5: parent erob70f__i_f_xx_18cx_v3_mc2a_9x_xx -> erob70f__i_f_xx_18cx_v3_mc2a_9x_xx_4
- joint revolute_6: origin xyz=-0.0204 3.46945e-17 4.68375e-17 rpy=-5.20761e-16 -1.22145e-16 -1.5708 -> xyz=-0.0204 -2.59021e-09 1.9082e-15 rpy=-4.89048e-16 2.36725e-16 -1.5708; parent erob70f__i_f_xx_18cx_v3_mc2a_9x_xx_7 -> erob70f__i_f_xx_18cx_v3_mc2a_9x_xx_8
